File: circuits/Legacy.brd (EAGLE design)
At the start: 42.9 x 68.6 mm, 17 parts, among them Y1 16MHz

Commit message: updated circuit schematics
Parts:
- removed J1: (no value), 001_SparkFun-Connectors:1X04
Connections:
- net 3.3V: no longer J1.2
- net 5V: no longer J1.1
- net N$12: no longer J1.4
- net N$5: no longer J1.3
Routing:
- net N$12: track 94.5 -> 12.1 mm
- net N$5: track 81.6 -> 9.18 mm
- net 3.3V: track 236.3 -> 210.6 mm
- net 5V: track 155.9 -> 130.3 mm
- net N$4: track 63.6 -> 71.4 mm
- net N$7: track 48.3 -> 54.5 mm
- net N$11: track 23.9 -> 27.3 mm
- net N$2: track 29.4 -> 30.1 mm
- net N$3: track 23.6 -> 24.1 mm
- net N$15: track 51.7 -> 51.2 mm, vias 1 -> 0
Other:
- board text removed: "GND"
- board text removed: "SCL"
- board text removed: "SDA"
- board text removed: "VCC"
