File: circuits/Legacy.sch (EAGLE design)
At the start: 17 parts, among them Y1 16MHz

Commit message: updated circuit schematics
Parts:
- removed J1: (no value), 001_SparkFun-Connectors:M04PTH
Connections:
- net 3.3V: no longer J1.2
- net 5V: no longer J1.1
- net N$12: no longer J1.4
- net N$5: no longer J1.3
Changed lines of the file:
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@@
 <?xml version="1.0" encoding="utf-8"?>
 <!DOCTYPE eagle SYSTEM "eagle.dtd">
-<eagle version="8.5.2">
+<eagle version="9.1.3">
 <drawing>
 <settings>
@@
 <part name="GND6" library="001_SparkFun-Aesthetics" deviceset="GND2" device=""/>
 <part name="GND7" library="001_SparkFun-Aesthetics" deviceset="GND2" device=""/>
-<part name="J1" library="001_SparkFun-Connectors" deviceset="M04" device="PTH"/>
-<part name="SUPPLY8" library="001_SparkFun-Aesthetics" deviceset="5V" device=""/>
-<part name="GND8" library="001_SparkFun-Aesthetics" deviceset="GND2" device=""/>
 </parts>
 <sheets>
@@
 <instance part="GND6" gate="G$1" x="152.4" y="0"/>
 <instance part="GND7" gate="G$1" x="175.26" y="0"/>
-<instance part="J1" gate="G$1" x="162.56" y="91.44" rot="R180"/>
-<instance part="SUPPLY8" gate="G$1" x="154.94" y="111.76"/>
-<instance part="GND8" gate="G$1" x="154.94" y="50.8"/>
 </instances>
 <busses>
@@
 <wire x1="210.82" y1="91.44" x2="210.82" y2="101.6" width="0.1524" layer="91"/>
 <wire x1="210.82" y1="101.6" x2="147.32" y2="101.6" width="0.1524" layer="91"/>
-<wire x1="147.32" y1="101.6" x2="147.32" y2="88.9" width="0.1524" layer="91"/>
-<wire x1="147.32" y1="88.9" x2="147.32" y2="83.82" width="0.1524" layer="91"/>
+<wire x1="147.32" y1="101.6" x2="147.32" y2="83.82" width="0.1524" layer="91"/>
 <wire x1="147.32" y1="83.82" x2="71.12" y2="83.82" width="0.1524" layer="91"/>
 <wire x1="71.12" y1="83.82" x2="71.12" y2="63.5" width="0.1524" layer="91"/>
 <pinref part="MICROCONTROLER" gate="G$1" pin="PC4(ADC4/SDA)"/>
 <wire x1="71.12" y1="63.5" x2="68.58" y2="63.5" width="0.1524" layer="91"/>
-<pinref part="J1" gate="G$1" pin="3"/>
-<wire x1="157.48" y1="88.9" x2="147.32" y2="88.9" width="0.1524" layer="91"/>
-<junction x="147.32" y="88.9"/>
 </segment>
 </net>
@@
 <wire x1="73.66" y1="60.96" x2="73.66" y2="81.28" width="0.1524" layer="91"/>
 <wire x1="73.66" y1="81.28" x2="152.4" y2="81.28" width="0.1524" layer="91"/>
-<wire x1="152.4" y1="81.28" x2="152.4" y2="86.36" width="0.1524" layer="91"/>
-<wire x1="152.4" y1="86.36" x2="152.4" y2="99.06" width="0.1524" layer="91"/>
+<wire x1="152.4" y1="81.28" x2="152.4" y2="99.06" width="0.1524" layer="91"/>
 <wire x1="152.4" y1="99.06" x2="213.36" y2="99.06" width="0.1524" layer="91"/>
 <wire x1="213.36" y1="99.06" x2="213.36" y2="88.9" width="0.1524" layer="91"/>
 <pinref part="SINGLE_BOARD_COMPUTER" gate="G$1" pin="SCL"/>
 <wire x1="213.36" y1="88.9" x2="208.28" y2="88.9" width="0.1524" layer="91"/>
-<pinref part="J1" gate="G$1" pin="4"/>
-<wire x1="157.48" y1="86.36" x2="152.4" y2="86.36" width="0.1524" layer="91"/>
-<junction x="152.4" y="86.36"/>
 </segment>
 </net>
@@
 <junction x="175.26" y="91.44"/>
 <pinref part="SUPPLY7" gate="G$1" pin="5V"/>
-</segment>
-<segment>
-<pinref part="J1" gate="G$1" pin="1"/>
-<wire x1="154.94" y1="93.98" x2="157.48" y2="93.98" width="0.1524" layer="91"/>
-<wire x1="154.94" y1="111.76" x2="154.94" y2="93.98" width="0.1524" layer="91"/>
-<pinref part="SUPPLY8" gate="G$1" pin="5V"/>
 </segment>
 </net>
@@
 <pinref part="GND1" gate="G$1" pin="3.3V"/>
 </segment>
-<segment>
-<pinref part="J1" gate="G$1" pin="2"/>
-<wire x1="157.48" y1="91.44" x2="154.94" y2="91.44" width="0.1524" layer="91"/>
-<wire x1="154.94" y1="91.44" x2="154.94" y2="53.34" width="0.1524" layer="91"/>
-<pinref part="GND8" gate="G$1" pin="3.3V"/>
-</segment>
-</net>
+</net>
